File: pcbs/centrall_microcontroller/centrall_microcontroller.kicad_sch (KiCad schematic)
At the start: 36 parts, among them Q1 BS170F, Q2 BS170F, SW1 Reset, U2 Pico, U3 L7805, U4 LM2596S-ADJ

Commit message: values change
Parts:
- R2: value 5K -> 1K
- RV1: value W103 (10K) -> W203 (20K)
Changed lines of the file:
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@@
 			)
 		)
-		(property "Value" "W103 (10K)"
+		(property "Value" "W203 (20K)"
 			(at 193.04 19.05 90)
 			(effects
@@
 			)
 		)
-		(property "Value" "5K"
+		(property "Value" "1K"
 			(at 170.18 19.05 90)
 			(effects
