File: pcbs/drill_pcb/drill_pcb.kicad_sch (KiCad schematic)
At the start: 26 parts, among them J1 24V IN, J10 WEIGHT SENSOR, J11 STEPPER STORAGE, J2 DC MOTOR 24 V, J3 DC MOTOR UART, J4 ENCODER VERTICAL DRIVE, J5 LIMIT SENSOR TOP, J6 HEIGHT SENSOR, J7 STEPPER VERTICAL DRIVE, J8 ENCODER STORAGE, J9 LIMIT SENSOR BOTTOM, U1 ESP32-DevKitC, U2 LM3940

Commit message: Cloned last version of PCB to preserve documentation for already manufactured hardware. New version of PCB includes connector for surface sample weighing, UART0 JST connector, I2C pullup resistors, new fuse footprint
Parts:
- added J12: SURFACE WEIGHT SENSOR, Connector_JST:JST_XH_B7B-XH-A_1x07_P2.50mm_Vertical, symbol Connector:Screw_Terminal_01x07
- added J13: uC COMMUNICATION, Connector_JST:JST_XH_B3B-XH-A_1x03_P2.50mm_Vertical, symbol Connector:Screw_Terminal_01x03
- added R2, R3: 2200, Resistor_SMD:R_1206_3216Metric, symbol Device:R
- F1, F2: footprint drill_fuseHolderATO:fuseHolderATO -> drill_fuseHolderATO:AUTOFUSE_HOLDER
- J10: value WEIGHT SENSOR -> DEEP WEIGHT SENSOR
Connections:
- net +3.3V: now also J12.2 (Pin_2), R2.2, R3.2
- net +5V: now also J12.1 (Pin_1)
- net GND: now also J12.7 (Pin_7), J13.1 (Pin_1)
- net SCL1: now also J12.3 (Pin_3), R3.1
- net SDA1: now also J12.4 (Pin_4), R2.1
- net RX0: now reaches U1.34 (U0RXD/GPIO3)
- net RX0: now also J13.3 (Pin_3)
- net TX0: now reaches U1.35 (U0TXD/GPIO1)
- net TX0: now also J13.2 (Pin_2)
- net ADC_DRDY renamed ADC_DEEP_DRDY
- net ADC_RST renamed ADC_DEEP_RST
- new net ADC_SURF_DRDY: J12.5 (Pin_5)
- new net ADC_SURF_RST: J12.6 (Pin_6)
- no-connect marks 15 -> 13

Commit message: pcb changes, code changes
Parts:
- added C8: 0.1 μF, symbol Device:C
- added R4: R, symbol Device:R
- added U3: INA219BxD, Package_SO:SOIC-8_3.9x4.9mm_P1.27mm, symbol Sensor_Energy:INA219BxD
Connections:
- net +3.3V: now also C8.1, U3.5 (VS)
- net GND: now also C8.2, U3.6 (GND)
- net SCL1: now also U3.4 (SCL)
- net SDA1: now also U3.3 (SDA)
- net DRVR_STORAGE_0: no longer names the net of A2.17 (DIAG0)
- net DRVR_STORAGE_0: no longer U1.6 (VDET_2/GPIO35/ADC1_CH7)
- net DRVR_STORAGE_1: no longer names the net of A2.18 (DIAG1)
- net DRVR_STORAGE_1: no longer U1.5 (VDET_1/GPIO34/ADC1_CH6)
- no-connect marks 13 -> 15
